File: PCB_impedance/PCB_impedance.kicad_sch (KiCad schematic)
At the start: 49 parts, among them J1 Screw_Terminal_01x04, J2 Conn_02x20_Odd_Even, J3 Screw_Terminal_01x04, J4 Screw_Terminal_01x04, J5 Screw_Terminal_01x04, U1 CD74HC4067M, U2 CD74HC4067M, U3 CD74HC4067M, U4 CD74HC4067M, U6 AD5941, U7 MCP1727-3302xMF

Commit message: Correction to the PCB schematic for measuring impedance (replacement of the multiplexer and add new connector for electrodes)
Parts:
- removed C1, C3, C5, C7: 10u, Capacitor_SMD:C_0805_2012Metric, symbol Device:C
- removed C2, C4, C6, C8: 100n, Capacitor_SMD:C_0805_2012Metric, symbol Device:C
- removed J1, J3, J4, J5: Screw_Terminal_01x04, AAA_MAZZA_project:TerminalBlock_MetzConnect_Type059_RT06304HBWC_1x04_P3.50mm_Horizontal, symbol Connector:Screw_Terminal_01x04
- removed U1, U2, U3, U4: CD74HC4067M, Package_SO:SOIC-24W_7.5x15.4mm_P1.27mm, symbol 74xx:CD74HC4067M
- added C33, C36, C38, C40: 10u, Capacitor_SMD:C_0805_2012Metric, symbol Device:C
- added C34, C35, C37, C39: 100n, Capacitor_SMD:C_0805_2012Metric, symbol Device:C
- added J6: Conn_01x16_Socket, lib_mesure_impedance:conn_1x16_PPPC082LFBN-RC, symbol Connector:Conn_01x16_Socket
- added U1, U2, U3, U4: ADG706BRUZ-REEL, lib_mesure_impedance:ADG706BRUZ, symbol lib_mesure_impedance:ADG706BRUZ-REEL
- R3: footprint (none) -> Resistor_SMD:R_0805_2012Metric; Digikey Part Number (none) -> YAG4820DKR-ND; Manufacturer (none) -> YAGEO; Manufacturer Part Number (none) -> RT0805BRD0710RL
- R4: footprint (none) -> Resistor_SMD:R_0805_2012Metric; Digikey Part Number (none) -> YAG1763DKR-ND; Manufacturer (none) -> YAGEO; Manufacturer Part Number (none) -> RT0805BRD0710KL
- R5, R6: footprint (none) -> Resistor_SMD:R_0805_2012Metric; Digikey Part Number (none) -> 13-RC0805FR-131KLDKR-ND; Manufacturer (none) -> YAGEO; Manufacturer Part Number (none) -> RC0805FR-131KL
- R7, R8: footprint (none) -> Resistor_SMD:R_0805_2012Metric; Digikey Part Number (none) -> 311-0.0ARDKR-ND; Manufacturer (none) -> YAGEO; Manufacturer Part Number (none) -> RC0805JR-070RL
- U6: footprint AAA_MAZZA_project:AD5941_footprint -> lib_mesure_impedance:AD5941_footprint
Connections:
- net +3V3: now also C33.1, C34.1, C35.1, C36.1, C37.1, C38.1, C39.1, C40.1, U1.1 (VDD), U2.1 (VDD), U3.1 (VDD), U4.1 (VDD)
- net E1: now also J6.1 (Pin_1), U1.19 (S1), U2.19 (S1), U3.19 (S1), U4.19 (S1)
- net E10: now also J6.10 (Pin_10), U1.10 (S10), U2.10 (S10), U3.10 (S10), U4.10 (S10)
- net E11: now also J6.11 (Pin_11), U1.9 (S11), U2.9 (S11), U3.9 (S11), U4.9 (S11)
- net E12: now also J6.12 (Pin_12), U1.8 (S12), U2.8 (S12), U3.8 (S12), U4.8 (S12)
- net E13: now also J6.13 (Pin_13), U1.7 (S13), U2.7 (S13), U3.7 (S13), U4.7 (S13)
- net E14: now also J6.14 (Pin_14), U1.6 (S14), U2.6 (S14), U3.6 (S14), U4.6 (S14)
- net E15: now also J6.15 (Pin_15), U1.5 (S15), U2.5 (S15), U3.5 (S15), U4.5 (S15)
- net E2: now also J6.2 (Pin_2), U1.20 (S2), U2.20 (S2), U3.20 (S2), U4.20 (S2)
- net E3: now also J6.3 (Pin_3), U1.21 (S3), U2.21 (S3), U3.21 (S3), U4.21 (S3)
- net E4: now also J6.4 (Pin_4), U1.22 (S4), U2.22 (S4), U3.22 (S4), U4.22 (S4)
- net E5: now also J6.5 (Pin_5), U1.23 (S5), U2.23 (S5), U3.23 (S5), U4.23 (S5)
- net E6: now also J6.6 (Pin_6), U1.24 (S6), U2.24 (S6), U3.24 (S6), U4.24 (S6)
- net E7: now also J6.7 (Pin_7), U1.25 (S7), U2.25 (S7), U3.25 (S7), U4.25 (S7)
- net E8: now also J6.8 (Pin_8), U1.26 (S8), U2.26 (S8), U3.26 (S8), U4.26 (S8)
- net E9: now also J6.9 (Pin_9), U1.11 (S9), U2.11 (S9), U3.11 (S9), U4.11 (S9)
- net F+: now also U4.28 (D)
- net F-: now also U3.28 (D)
- net GND: now also C33.2, C34.2, C35.2, C36.2, C37.2, C38.2, C39.2, C40.2, U1.12 (GND), U1.27 (VSS), U2.12 (GND), U2.27 (VSS), U3.12 (GND), U3.27 (VSS), U4.12 (GND), U4.27 (VSS)
- net MUX_S0: now also J2.15 (Pin_15), U4.17 (A0); no longer J2.27 (Pin_27)
- net MUX_S1: now also J2.17 (Pin_17), U4.16 (A1); no longer J2.29 (Pin_29)
- net MUX_S2: now also J2.27 (Pin_27), U4.15 (A2); no longer J2.31 (Pin_31)
- net MUX_S3: now also J2.29 (Pin_29), U4.14 (A3); no longer J2.33 (Pin_33)
- net S+: now also U2.28 (D)
- net S-: now also U1.28 (D)
- net at C9.1, U6.5 (AVDD_REG): no longer C10.1, U6.14 (DVDD_REG_1V8)
- net MUX_S8: now reaches J2.16 (Pin_16)
- net MUX_S8: now also U2.17 (A0)
- net MUX_S9: now reaches J2.18 (Pin_18)
- net MUX_S9: now also U2.16 (A1)
- net MUX_S10: now reaches J2.22 (Pin_22)
- net MUX_S10: now also U2.15 (A2)
- net MUX_S11: now reaches J2.26 (Pin_26)
- net MUX_S11: now also U2.14 (A3)
- net MUX_S12: now reaches J2.28 (Pin_28)
- net MUX_S12: now also U1.17 (A0)
- net MUX_S13: now reaches J2.32 (Pin_32)
- net MUX_S13: now also U1.16 (A1)
- net MUX_S6: now reaches J2.35 (Pin_35)
- net MUX_S6: now also U3.15 (A2)
- net MUX_S14: now reaches J2.36 (Pin_36)
- net MUX_S14: now also U1.15 (A2)
- net MUX_S7: now reaches J2.37 (Pin_37)
- net MUX_S7: now also U3.14 (A3)
- net MUX_S15: now reaches J2.38 (Pin_38)
- net MUX_S15: now also U1.14 (A3)
- net MUX_En0 renamed MUX_EN0
- net MUX_EN0: now also U4.18 (EN)
- net MUX_En1 renamed MUX_EN1
- net MUX_EN1: now also U3.18 (EN)
- net MUX_En2 renamed MUX_EN2
- net MUX_EN2: now also U2.18 (EN)
- net MUX_En3 renamed MUX_EN3
- net MUX_EN3: now also U1.18 (EN)
- new net: C10.1, U6.14 (DVDD_REG_1V8)
- new net: U4.13 (NC), U4.2 (NC), U4.3 (NC)
- new net: U2.13 (NC), U2.2 (NC), U2.3 (NC)
- new net: U1.13 (NC), U1.2 (NC), U1.3 (NC)
- new net: U3.13 (NC), U3.2 (NC), U3.3 (NC)
- new net E16: J6.16 (Pin_16), U1.4 (S16), U2.4 (S16), U3.4 (S16), U4.4 (S16)
- new net MUX_S4: J2.31 (Pin_31), U3.17 (A0)
- new net MUX_S5: J2.33 (Pin_33), U3.16 (A1)
- no-connect marks 25 -> 17
Other:
- note added: "A precision external resistor Rcal is required to calibrate DAC. Recommanded value : 10k"
- note added: "The ADG706 switches one of 16 inputs (S1-S16) to a common output, D, as determined by the 4-bit binary address lines A0, A1, A2, and A3"
- note added: "U1 Decoupling capacitors"
- note added: "U2 Decoupling capacitors"
- note added: "U3 Decoupling capacitors"
- note added: "U4 Decoupling capacitors"
- note removed: "A precision external resistor Rcal is required to calibrate DAC"
- moved on the sheet: C10, C9, R4

Commit message: Multiplexer routing complete
Parts:
- removed C33, C36, C38, C40: 10u, Capacitor_SMD:C_0805_2012Metric, symbol Device:C
- removed C34, C35, C37, C39: 100n, Capacitor_SMD:C_0805_2012Metric, symbol Device:C
- removed U1, U2, U3, U4: ADG706BRUZ-REEL, lib_mesure_impedance:ADG706BRUZ, symbol lib_mesure_impedance:ADG706BRUZ-REEL
- added C1, C3, C5, C7: 100n, Capacitor_SMD:C_0603_1608Metric, symbol Device:C
- added C2, C4, C6, C8: 10u, Capacitor_SMD:C_0603_1608Metric, symbol Device:C
- added H1, H2, H3, H4: MountingHole, MountingHole:MountingHole_2.7mm_Pad, symbol Mechanical:MountingHole
- added J1: Conn_01x16_Socket, symbol Connector:Conn_01x16_Socket
- added U1, U2, U3, U5: ADG726BSUZ, lib_mesure_impedance:ADG726SBUZ, symbol lib_mesure_impedance:ADG726BSUZ
- J2: footprint Connector_PinHeader_2.54mm:PinHeader_2x20_P2.54mm_Vertical -> lib_mesure_impedance:PinHeader_2x20_P2.54mm_Vertical
Connections:
- net MUX_S0 is gone; now on net MUX_EN1: J2.15 (Pin_15)
- net MUX_S2 is gone; now on net MUX_EN2: J2.27 (Pin_27)
- net MUX_S3 is gone; now on net MUX_EN3: J2.29 (Pin_29)
- net +3V3: now also C1.1, C2.1, C3.1, C4.1, C5.1, C6.1, C7.1, C8.1, U1.13 (VDD), U1.14 (VDD), U1.20 (CSB*), U2.13 (VDD), U2.14 (VDD), U2.20 (CSB*), U3.13 (VDD), U3.14 (VDD), U3.20 (CSB*), U5.13 (VDD), U5.14 (VDD), U5.20 (CSB*)
- net E1: now also U1.12 (S1A), U2.12 (S1A), U3.12 (S1A), U5.12 (S1A)
- net E10: now also U1.3 (S10A), U2.3 (S10A), U3.3 (S10A), U5.3 (S10A)
- net E11: now also U1.2 (S11A), U2.2 (S11A), U3.2 (S11A), U5.2 (S11A)
- net E12: now also U1.1 (S12A), U2.1 (S12A), U3.1 (S12A), U5.1 (S12A)
- net E13: now also U1.48 (S13A), U2.48 (S13A), U3.48 (S13A), U5.48 (S13A)
- net E14: now also U1.47 (S14A), U2.47 (S14A), U3.47 (S14A), U5.47 (S14A)
- net E15: now also U1.46 (S15A), U2.46 (S15A), U3.46 (S15A), U5.46 (S15A)
- net E16: now also U1.45 (S16A), U2.45 (S16A), U3.45 (S16A), U5.45 (S16A)
- net E2: now also U1.11 (S2A), U2.11 (S2A), U3.11 (S2A), U5.11 (S2A)
- net E3: now also U1.10 (S3A), U2.10 (S3A), U3.10 (S3A), U5.10 (S3A)
- net E4: now also U1.9 (S4A), U2.9 (S4A), U3.9 (S4A), U5.9 (S4A)
- net E5: now also U1.8 (S5A), U2.8 (S5A), U3.8 (S5A), U5.8 (S5A)
- net E6: now also U1.7 (S6A), U2.7 (S6A), U3.7 (S6A), U5.7 (S6A)
- net E7: now also U1.6 (S7A), U2.6 (S7A), U3.6 (S7A), U5.6 (S7A)
- net E8: now also U1.5 (S8A), U2.5 (S8A), U3.5 (S8A), U5.5 (S8A)
- net E9: now also U1.4 (S9A), U2.4 (S9A), U3.4 (S9A), U5.4 (S9A)
- net F+: now also U5.43 (DA)
- net F-: now also U2.43 (DA)
- net GND: now also C1.2, C2.2, C3.2, C4.2, C5.2, C6.2, C7.2, C8.2, U1.23 (GND), U1.24 (VSS), U2.23 (GND), U2.24 (VSS), U3.23 (GND), U3.24 (VSS), U5.23 (GND), U5.24 (VSS)
- net MUX_EN0: now also J2.13 (Pin_13), U5.22 (EN*); no longer J2.5 (Pin_5)
- net MUX_EN1: now also U1.22 (EN*); no longer J2.7 (Pin_7)
- net MUX_EN2: now also U2.22 (EN*); no longer J2.11 (Pin_11)
- net MUX_EN3: now also U3.22 (EN*); no longer J2.13 (Pin_13)
- net S+: now also U1.43 (DA)
- net S-: now also U3.43 (DA)
- net F+_node: now reaches C29.1, R5.2
- net S-_node: now reaches C32.2, R8.2
- net S+_node: now reaches C31.2, R7.2
- net F-_node: now reaches C30.2, R6.2
- net MUX_CSA3: now reaches J2.40 (Pin_40)
- net MUX_CSA3: now also U3.19 (CSA*)
- net MUX_S1: no longer names the net of J2.17 (Pin_17)
- net MUX_S10 renamed MUX_WR1
- net MUX_WR1: now also U1.21 (WR*)
- net MUX_S11 renamed MUX_WR2
- net MUX_WR2: now also U2.21 (WR*)
- net MUX_S12 renamed MUX_WR3
- net MUX_WR3: now also U3.21 (WR*)
- net MUX_S13 renamed MUX_CSA0
- net MUX_CSA0: now also U5.19 (CSA*)
- net MUX_S14 renamed MUX_CSA1
- net MUX_CSA1: now also U1.19 (CSA*)
- net MUX_S15 renamed MUX_CSA2
- net MUX_CSA2: now also U2.19 (CSA*)
- net MUX_S4 renamed MUX_A0
- net MUX_A0: now also U1.15 (A0), U2.15 (A0), U3.15 (A0), U5.15 (A0)
- net MUX_S5 renamed MUX_A1
- net MUX_A1: now also U1.16 (A1), U2.16 (A1), U3.16 (A1), U5.16 (A1)
- net MUX_S6 renamed MUX_A2
- net MUX_A2: now also U1.17 (A2), U2.17 (A2), U3.17 (A2), U5.17 (A2)
- net MUX_S7 renamed MUX_A3
- net MUX_A3: now also U1.18 (A3), U2.18 (A3), U3.18 (A3), U5.18 (A3)
- net MUX_S8: no longer names the net of J2.16 (Pin_16)
- net MUX_S9 renamed MUX_WR0
- net MUX_WR0: now also U5.21 (WR*)
- no-connect marks 17 -> 93
Other:
- note added: "U5 Decoupling capacitors"
- note removed: "TODO PCB : 1) Assigner et controler les footprint 2) Review Schematic"
- note removed: "The ADG706 switches one of 16 inputs (S1-S16) to a common output, D, as determined by the 4-bit binary address lines A0, A1, A2, and A3"
- note removed: "U4 Decoupling capacitors"
- moved on the sheet: C10, C14, C15, C16, C17, C18, C19, C20, C21, C22, C23, C24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
