File: PCB_impedance/PCB_impedance.kicad_sch (KiCad schematic)
At the start: 51 parts, among them J1 Conn_01x16_Socket, J2 Conn_02x20_Odd_Even, J6 Conn_01x16_Socket, U1 ADG726BSUZ, U2 ADG726BSUZ, U3 ADG726BSUZ, U5 ADG726BSUZ, U6 AD5941, U7 MCP1727-3302xMF

Commit message: PCB routing with the AD5940 is complete
Parts:
- removed J1: Conn_01x16_Socket, symbol Connector:Conn_01x16_Socket
- J2: footprint lib_mesure_impedance:PinHeader_2x20_P2.54mm_Vertical -> Connector_PinSocket_2.54mm:PinSocket_2x20_P2.54mm_Vertical; Digikey Part Number S6104-ND -> (none); Manufacturer Sullins Connector Solutions -> (none); Manufacturer Part Number PPTC202LFBN-RC -> (none)
Other:
- note added: "For 3x3DFN package, the maximum package power dissipation at 60°C ambiant temperature is : P_D(max) = (125°C - 60°C) / 41°C/W = 1.585W"
- note added: "P_LDO = (5V - 3.3V) * (10mA (AD5940) + 4*5uA (ADG726)) = 0.02W"
- note added: "Power Dissipation"
- note added: "The maximum continuous junction temperature T_J(max) must stay under 125°C T_J(max) = P_LDO * Rtheta_JA + Tambiant = 0.02W * 41.0°C/W + 60°C = 60.7°C"
Changed lines of the file:
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@@
 		)
 	)
+	(text "For 3x3DFN package, the maximum package power dissipation at 60°C ambiant temperature is :\nP_D(max) = (125°C - 60°C) / 41°C/W = 1.585W"
+		(exclude_from_sim no)
+		(at 75.946 69.088 0)
+		(effects
+			(font
+				(size 0.762 0.762)
+				(thickness 0.1524)
+				(bold yes)
+			)
+			(justify left)
+		)
+	)
 	(text "Electrodes for 4-Wire Impedance Measurement \n(CE0, AIN2, AIN3, AIN1)"
 		(exclude_from_sim no)
@@
 		)
 	)
+	(text "P_LDO = (5V - 3.3V) * (10mA (AD5940) + 4*5uA (ADG726)) = 0.02W"
+		(exclude_from_sim no)
+		(at 75.946 73.406 0)
+		(effects
+			(font
+				(size 0.762 0.762)
+				(thickness 0.1588)
+			)
+			(justify left)
+		)
+	)
+	(text "The maximum continuous junction temperature T_J(max) must stay under 125°C\nT_J(max) = P_LDO * Rtheta_JA + Tambiant = 0.02W * 41.0°C/W + 60°C = 60.7°C"
+		(exclude_from_sim no)
+		(at 75.946 76.962 0)
+		(effects
+			(font
+				(size 0.762 0.762)
+				(thickness 0.1524)
+				(bold yes)
+			)
+			(justify left)
+		)
+	)
 	(text "CTIA and RTIA"
 		(exclude_from_sim no)
@@
 		)
 	)
+	(text "Power Dissipation"
+		(exclude_from_sim no)
+		(at 87.884 65.278 0)
+		(effects
+			(font
+				(size 1.778 1.778)
+				(thickness 0.254)
+				(bold yes)
+			)
+		)
+	)
 	(text "U5 Decoupling capacitors"
 		(exclude_from_sim no)
@@
 	)
 	(symbol
-		(lib_id "Connector:Conn_01x16_Socket")
-		(at 455.676 59.436 0)
-		(unit 1)
-		(exclude_from_sim no)
-		(in_bom yes)
-		(on_board yes)
-		(dnp no)
-		(fields_autoplaced yes)
-		(property "Reference" "J1"
-			(at 457.2 59.4359 0)
-			(effects
-				(font
-					(size 1.27 1.27)
-				)
-				(justify left)
-			)
-		)
-		(property "Value" "Conn_01x16_Socket"
-			(at 457.2 61.9759 0)
-			(effects
-				(font
-					(size 1.27 1.27)
-				)
-				(justify left)
-			)
-		)
-		(property "Footprint" ""
-			(at 455.676 59.436 0)
-			(effects
-				(font
-					(size 1.27 1.27)
-				)
-				(hide yes)
-			)
-		)
-		(property "Datasheet" "~"
-			(at 455.676 59.436 0)
-			(effects
-				(font
-					(size 1.27 1.27)
-				)
-				(hide yes)
-			)
-		)
-		(property "Description" "Generic connector, single row, 01x16, script generated"
-			(at 455.676 59.436 0)
-			(effects
-				(font
-					(size 1.27 1.27)
-				)
-				(hide yes)
-			)
-		)
-		(pin "16"
-		)
-		(pin "9"
-		)
-		(pin "14"
-		)
-		(pin "3"
-		)
-		(pin "12"
-		)
-		(pin "4"
-		)
-		(pin "11"
-		)
-		(pin "13"
-		)
-		(pin "10"
-		)
-		(pin "5"
-		)
-		(pin "1"
-		)
-		(pin "6"
-		)
-		(pin "7"
-		)
-		(pin "2"
-		)
-		(pin "8"
-		)
-		(pin "15"
-		)
-		(instances
-			(project "PCB_impedance"
-				(path "/17c54b31-e408-4e08-a1dc-baf1e1ebfa28"
-					(reference "J1")
-					(unit 1)
-				)
-			)
-		)
-	)
-	(symbol
 		(lib_id "power:GND")
 		(at 49.53 245.618 0)
@@
 			)
 		)
-		(property "Footprint" "lib_mesure_impedance:PinHeader_2x20_P2.54mm_Vertical"
+		(property "Footprint" "Connector_PinSocket_2.54mm:PinSocket_2x20_P2.54mm_Vertical"
 			(at 48.26 61.976 0)
 			(effects
@@
 			)
 		)
-		(property "Datasheet" "https://mm.digikey.com/Volume0/opasdata/d220001/medias/docus/937/Female_Headers.100_DS.pdf"
+		(property "Datasheet" ""
 			(at 48.26 61.976 0)
 			(effects
@@
 			)
 		)
-		(property "Description" "40 Position Header Connector 0.100\" (2.54mm) Through Hole Tin"
+		(property "Description" ""
 			(at 48.26 61.976 0)
 			(effects
@@
 			)
 		)
-		(property "Manufacturer" "Sullins Connector Solutions"
+		(property "Manufacturer" ""
 			(at 48.26 61.976 0)
 			(effects
@@
 			)
 		)
-		(property "Manufacturer Part Number" "PPTC202LFBN-RC"
+		(property "Manufacturer Part Number" ""
 			(at 48.26 61.976 0)
 			(effects
@@
 			)
 		)
-		(property "Digikey Part Number" "S6104-ND"
+		(property "Digikey Part Number" ""
 			(at 48.26 61.976 0)
 			(effects
